Commit message: Tutlebot2+URG

File: trcp_description/robots/kobuki_hexagons_kinect.urdf.xacro (robot description, xacro)
@@ -6,5 +6,5 @@
 -->
 <robot name="turtlebot" xmlns:xacro="http://ros.org/wiki/xacro">
-  <xacro:include filename="$(find turtlebot_description)/urdf/turtlebot_library.urdf.xacro" />
+  <xacro:include filename="$(find trcp_description)/urdf/turtlebot_library.urdf.xacro" />
   <kobuki/>
   <stack_hexagons parent="base_link"/>

File: trcp_description/urdf/turtlebot_library.urdf.xacro (robot description, xacro)
@@ -5,15 +5,34 @@
 <robot xmlns:xacro="http://ros.org/wiki/xacro">
   <!-- General -->
-  <xacro:include filename="$(find turtlebot_description)/urdf/common_properties.urdf.xacro"/>
-  <xacro:include filename="$(find turtlebot_description)/urdf/turtlebot_properties.urdf.xacro"/>
+  <xacro:include filename="$(find trcp_description)/urdf/common_properties.urdf.xacro"/>
+  <xacro:include filename="$(find trcp_description)/urdf/turtlebot_properties.urdf.xacro"/>
   <!-- Bases -->
   <xacro:include filename="$(find create_description)/urdf/create.urdf.xacro"/>
   <xacro:include filename="$(find kobuki_description)/urdf/kobuki.urdf.xacro" />
   <!-- Stacks -->
-  <xacro:include filename="$(find turtlebot_description)/urdf/stacks/circles.urdf.xacro"/>
-  <xacro:include filename="$(find turtlebot_description)/urdf/stacks/hexagons.urdf.xacro"/>
+  <xacro:include filename="$(find trcp_description)/urdf/stacks/circles.urdf.xacro"/>
+  <xacro:include filename="$(find trcp_description)/urdf/stacks/hexagons.urdf.xacro"/>
   <!-- 3D Sensors -->
-  <xacro:include filename="$(find turtlebot_description)/urdf/sensors/kinect.urdf.xacro"/>
-  <xacro:include filename="$(find turtlebot_description)/urdf/sensors/asus_xtion_pro.urdf.xacro"/>
-<xacro:include filename="$(find trcp_description)/urdf/sensors/hokuyo.urdf.xacro"/>
+  <xacro:include filename="$(find trcp_description)/urdf/sensors/kinect.urdf.xacro"/>
+  <xacro:include filename="$(find trcp_description)/urdf/sensors/asus_xtion_pro.urdf.xacro"/>
+ <joint name="laser" type="fixed">
+    <origin xyz="-0.005 0.00 0.360" rpy="3.14159 0 0" />
+    <parent link="base_link" />
+    <child link="base_laser_link" />
+  </joint>
+  <link name="base_laser_link">
+    <visual>
+      <geometry>
+        <box size="0.05 0.05 0.07" />
+      </geometry>
+      <material name="Green" />
+    </visual>
+    <inertial>
+      <mass value="0.000001" />
+      <origin xyz="0 0 0" />
+      <inertia ixx="0.0001" ixy="0.0" ixz="0.0"
+        iyy="0.0001" iyz="0.0"
+        izz="0.0001" />
+    </inertial>
+  </link>
 </robot>

Commit message: tb2

File: trcp_description/robots/kobuki_hexagons_kinect.urdf.xacro (robot description, xacro)
@@ -10,3 +10,4 @@
   <stack_hexagons parent="base_link"/>
   <sensor_kinect  parent="base_link"/>
+  <sensor_hokuyo  parent="base_link"/>
 </robot>

File: trcp_description/urdf/turtlebot_library.urdf.xacro (robot description, xacro)
@@ -16,23 +16,4 @@
   <xacro:include filename="$(find trcp_description)/urdf/sensors/kinect.urdf.xacro"/>
   <xacro:include filename="$(find trcp_description)/urdf/sensors/asus_xtion_pro.urdf.xacro"/>
- <joint name="laser" type="fixed">
-    <origin xyz="-0.005 0.00 0.360" rpy="3.14159 0 0" />
-    <parent link="base_link" />
-    <child link="base_laser_link" />
-  </joint>
-  <link name="base_laser_link">
-    <visual>
-      <geometry>
-        <box size="0.05 0.05 0.07" />
-      </geometry>
-      <material name="Green" />
-    </visual>
-    <inertial>
-      <mass value="0.000001" />
-      <origin xyz="0 0 0" />
-      <inertia ixx="0.0001" ixy="0.0" ixz="0.0"
-        iyy="0.0001" iyz="0.0"
-        izz="0.0001" />
-    </inertial>
-  </link>
+  <xacro:include filename="$(find trcp_description)/urdf/sensors/hokuyo.urdf.xacro"/>
 </robot>
