Commit message: LRF

File: trcp_description/urdf/sensors/hokuyo.urdf.xacro (robot description, xacro)
@@ -24,5 +24,5 @@
  </link>
  <joint name="hokuyo_joint" type="fixed">
-   <origin xyz="0.10 0.0 0.13" rpy="0 0 0"/>
+   <origin xyz="0.132 0.0 0.13" rpy="3.14 0 0"/>
    <parent link="${parent}"/>
    <child link="laser_joint"/>

File: trcp_description/urdf/stacks/hexagons.urdf.xacro (robot description, xacro)
@@ -135,5 +135,8 @@
     <stack_bottom_pole parent="${parent}" number="5" x_loc="-0.055" y_loc="-0.120" z_loc="0.1028"/>
     <joint name="plate_bottom_joint" type="fixed">
-      <origin xyz="0.02364 0.0 0.1306" rpy="0 0 0"/>
+<!--
+      <origin xyz="0.02364 0.0 0.1307" rpy="0 0 0"/>
+-->
+      <origin xyz="0.02364 0.0 0.1507" rpy="0 0 0"/>
       <parent link="${parent}"/>
       <child link="plate_bottom_link"/>

Commit message: remote

File: trcp_description/urdf/sensors/hokuyo.urdf.xacro (robot description, xacro)
@@ -14,5 +14,5 @@
      <origin xyz="0 0 0" rpy="0 0 0"/>
      <geometry>
-<mesh filename="package://turtlebot_description/meshes/sensors/hokuyo.dae"/>
+<mesh filename="package://trcp_description/meshes/sensors/hokuyo.dae"/>
      </geometry>
    </visual>
